File: railroad-keyboard.sch (KiCad schematic (older format))
At the start: 66 parts

Commit message: First full schematic draft
Parts:
- added D? (x88): SOD-123, symbol Device:D_Small
- added MX? (x88): MX-NoLED, symbol MX_Alps_Hybrid:MX-NoLED
Connections:
- net labels added: ROW1, ROW2, ROW3, ROW4, ROW5, ROW6, ROW7, ROW8
- wire segments 102 -> 438
Other:
- moved on the sheet: R?

Commit message: Label D and MX in schematic
Parts:
- gave numbers to parts that had none: 226
