File: railroad-keyboard.sch (KiCad schematic (older format))
At the start: 229 parts, among them J1 1734510-1, J2 Conn_01x01, J3 Conn_01x01, SW1 SW_Push, U1 ATmega32U4-AU, Y1 16MHz

Commit message: Further alternate layouts WIP
Parts:
- added D700: SOD-123, Diode_SMD:D_SOD-123, symbol Device:D_Small
- added MX209_100: MX-NoLED, MX_Only:MXOnly-1U-NoLED, symbol MX_Alps_Hybrid:MX-NoLED
- added MX309_150: MX-NoLED, MX_Only:MXOnly-1.5U-NoLED, symbol MX_Alps_Hybrid:MX-NoLED
- added MX609_275, MX700_275: MX-NoLED, MX_Only:MXOnly-2.75U-NoLED, symbol MX_Alps_Hybrid:MX-NoLED
- added MX700_175: MX-NoLED, MX_Only:MXOnly-1.75U-NoLED, symbol MX_Alps_Hybrid:MX-NoLED
- MX601_100: renamed from MX601; footprint MX_Only:MXOnly-2.75U-NoLED -> MX_Only:MXOnly-1U-NoLED
- renumbered MX209 to MX209_150, MX309 to MX309_100, MX609 to MX609_175, MX708 to MX708_100
Connections:
- net COL0: now also MX700_175.1 (COL), MX700_275.1 (COL)
- net COL9: now also MX209_100.1 (COL), MX309_150.1 (COL), MX609_275.1 (COL)
- net ROW7: now also D700.1 (K)
- net at D209.2 (A), MX209_150.2 (ROW): now also MX209_100.2 (ROW)
- net at D309.2 (A), MX309_100.2 (ROW): now also MX309_150.2 (ROW)
- net at D609.2 (A), MX609_175.2 (ROW): now also MX609_275.2 (ROW)
- new net: D700.2 (A), MX700_175.2 (ROW), MX700_275.2 (ROW)
Other:
- moved on the sheet: D209, D309, D600, D609, D709

Commit message: miscellany
Parts:
- renumbered D0 to D1000, D100 to D1001, D500 to D1005, D1 to D1010, D101 to D1011, D2 to D1020, D102 to D1021, D3 to D1030, D103 to D1031, D4 to D1040, D104 to D1041, D5 to D1050, D105 to D1051, D6 to D1060, D106 to D1061, D7 to D1070, D107 to D1071, D8 to D1080, D108 to D1081, D9 to D1090, D109 to D1091, D10 to D1100, D210 to D1102, D200 to D2002, D300 to D2003, D201 to D2012, D301 to D2013, MX0 to MX1000, MX100_100 to MX1001_100, MX100_200 to MX1001_200, MX500_100 to MX1005_100, MX1 to MX1010, MX101 to MX1011, MX2 to MX1020, MX102 to MX1021, MX3 to MX1030, MX103 to MX1031, MX4 to MX1040, MX104 to MX1041, MX5 to MX1050, MX105 to MX1051, MX6 to MX1060, MX106 to MX1061, MX7 to MX1070, MX107 to MX1071, MX8 to MX1080, MX108 to MX1081, MX9_100 to MX1090_100, MX9_200 to MX1090_200, MX109 to MX1091, MX10 to MX1100, MX210_100 to MX1102_100, MX200 to MX2002, MX300 to MX2003, MX201 to MX2012, MX301 to MX2013
