File: railroad-keyboard-fullsize.sch (KiCad schematic (older format))
At the start: 208 parts, among them SW1 SW_Push, U1 ATmega32U4-AU, Y1 16MHz

Commit message: Divide into TKL and fullsize, annotate
Parts:
- added D011, D012, D110, D111, D211, D212, D310, D311, D411, D510, D511, D611, D612, D710, D711, D910, D911: SOD-123, symbol Device:D_Small
- added MX011, MX012, MX110, MX111, MX211, MX212, MX310, MX311, MX411, MX510, MX511, MX611, MX612, MX710, MX711, MX910, MX911: MX-NoLED, symbol MX_Alps_Hybrid:MX-NoLED
- C?: renamed from C3; footprint Diode_SMD:D_SOD-123 -> (none)
- C?: renamed from C7; footprint Diode_SMD:D_SOD-123 -> (none)
- C?: renamed from C6; footprint Diode_SMD:D_SOD-123 -> (none)
- C?: renamed from C5; footprint Diode_SMD:D_SOD-123 -> (none)
- C?: renamed from C4; footprint Diode_SMD:D_SOD-123 -> (none)
- C?: renamed from C1; footprint Diode_SMD:D_SOD-123 -> (none)
- C?: renamed from C2; footprint Diode_SMD:D_SOD-123 -> (none)
- D000: renamed from D0; footprint Diode_SMD:D_SOD-123 -> (none)
- D001: renamed from D1; footprint Diode_SMD:D_SOD-123 -> (none)
- D002: renamed from D2; footprint Diode_SMD:D_SOD-123 -> (none)
- D003: renamed from D3; footprint Diode_SMD:D_SOD-123 -> (none)
- D004: renamed from D4; footprint Diode_SMD:D_SOD-123 -> (none)
- D005: renamed from D5; footprint Diode_SMD:D_SOD-123 -> (none)
- D006: renamed from D6; footprint Diode_SMD:D_SOD-123 -> (none)
- D007: renamed from D7; footprint Diode_SMD:D_SOD-123 -> (none)
- D008: renamed from D8; footprint Diode_SMD:D_SOD-123 -> (none)
- D009: renamed from D9; footprint Diode_SMD:D_SOD-123 -> (none)
- D010: renamed from D10; footprint Diode_SMD:D_SOD-123 -> (none)
- D100, D101, D102, D103, D104, D105, D106, D107, D108, D109, D200, D201, D202, D203, D204, D205, D206, D207, D208, D209, D300, D301, D302, D303, D304, D305, D306, D307, D308, D309, D400, D401, D402, D403, D404, D405, D406, D407, D408, D409, D410, D501, D502, D503, D504, D505, D506, D507, D508, D509, D600, D601, D602, D603, D604, D605, D606, D607, D608, D609, D701, D702, D703, D704, D705, D706, D707, D708, D709, D800, D801, D802, D808, D809, D810, D900, D901, D902, D903, D904, D905, D906, D907, D908, D909: footprint Diode_SMD:D_SOD-123 -> (none)
- F?: renamed from F1; footprint Fuse:Fuse_1206_3216Metric -> (none)
- MX000: renamed from MX0; footprint MX_Alps_Hybrid:MX-1U-NoLED -> (none)
- MX001: renamed from MX1; footprint MX_Alps_Hybrid:MX-1U-NoLED -> (none)
- MX002: renamed from MX2; footprint MX_Alps_Hybrid:MX-1U-NoLED -> (none)
- MX003: renamed from MX3; footprint MX_Alps_Hybrid:MX-1U-NoLED -> (none)
- MX004: renamed from MX4; footprint MX_Alps_Hybrid:MX-1U-NoLED -> (none)
- MX005: renamed from MX5; footprint MX_Alps_Hybrid:MX-1U-NoLED -> (none)
- MX006: renamed from MX6; footprint MX_Alps_Hybrid:MX-1U-NoLED -> (none)
- MX007: renamed from MX7; footprint MX_Alps_Hybrid:MX-1U-NoLED -> (none)
- MX008: renamed from MX8; footprint MX_Alps_Hybrid:MX-1U-NoLED -> (none)
- MX009: renamed from MX9; footprint MX_Alps_Hybrid:MX-2U-NoLED -> (none)
- MX010: renamed from MX10; footprint MX_Alps_Hybrid:MX-1U-NoLED -> (none)
- MX100: footprint MX_Alps_Hybrid:MX-2U-NoLED -> (none)
- MX101, MX102, MX103, MX104, MX105, MX106, MX107, MX108, MX109, MX200, MX202, MX203, MX204, MX205, MX206, MX207, MX208, MX301, MX302, MX303, MX304, MX305, MX306, MX307, MX308, MX309, MX402, MX403, MX404, MX405, MX406, MX407, MX408, MX409, MX501, MX502, MX503, MX504, MX505, MX506, MX507, MX508, MX600, MX602, MX603, MX604, MX605, MX606, MX607, MX608, MX701, MX702, MX703, MX704, MX705, MX706, MX707, MX708, MX709, MX800, MX809, MX810, MX900, MX902, MX907, MX909: footprint MX_Alps_Hybrid:MX-1U-NoLED -> (none)
- MX201, MX209, MX300, MX801, MX808, MX908: footprint MX_Alps_Hybrid:MX-1.5U-NoLED -> (none)
- MX400, MX802, MX901: footprint MX_Alps_Hybrid:MX-1.25U-NoLED -> (none)
- MX401, MX905: footprint MX_Alps_Hybrid:MX-2.25U-NoLED -> (none)
- MX410: footprint MX_Alps_Hybrid:MX-ISO -> (none)
- MX509, MX609, MX903, MX906: footprint MX_Alps_Hybrid:MX-1.75U-NoLED -> (none)
- MX601, MX904: footprint MX_Alps_Hybrid:MX-2.75U-NoLED -> (none)
- R?: renamed from R4; footprint Resistor_SMD:R_0805_2012Metric -> (none)
- R?: renamed from R2; footprint Resistor_SMD:R_0805_2012Metric -> (none)
- R?: renamed from R3; footprint Resistor_SMD:R_0805_2012Metric -> (none)
- R?: renamed from R1; footprint Resistor_SMD:R_0805_2012Metric -> (none)
- SW?: renamed from SW1; footprint random-keyboard-parts:SKQG-1155865 -> (none)
- USB?: renamed from USB1; footprint random-keyboard-parts:Molex-0548190589 -> (none)
- Y?: renamed from Y1; footprint Crystal:Crystal_SMD_3225-4Pin_3.2x2.5mm -> (none)
- renumbered U1 to U?
Connections:
- net COL10: now also MX110.1 (COL), MX310.1 (COL), MX510.1 (COL), MX710.1 (COL), MX910.1 (COL)
- net ROW0: now also D011.1 (K), D012.1 (K)
- net ROW1: now also D110.1 (K), D111.1 (K)
- net ROW2: now also D211.1 (K), D212.1 (K)
- net ROW3: now also D310.1 (K), D311.1 (K)
- net ROW4: now also D411.1 (K)
- net ROW5: now also D510.1 (K), D511.1 (K)
- net ROW6: now also D611.1 (K), D612.1 (K)
- net ROW7: now also D710.1 (K), D711.1 (K)
- net ROW9: now also D910.1 (K), D911.1 (K)
- net COL12: now reaches U?.37 (PF6)
- net COL12: now also MX012.1 (COL), MX212.1 (COL), MX612.1 (COL)
- net COL11: now reaches U?.38 (PF5)
- net COL11: now also MX011.1 (COL), MX111.1 (COL), MX211.1 (COL), MX311.1 (COL), MX411.1 (COL), MX511.1 (COL), MX611.1 (COL), MX711.1 (COL), MX911.1 (COL)
- new net: D110.2 (A), MX110.2 (ROW)
- new net: D011.2 (A), MX011.2 (ROW)
- new net: D111.2 (A), MX111.2 (ROW)
- new net: D012.2 (A), MX012.2 (ROW)
- new net: D310.2 (A), MX310.2 (ROW)
- new net: D211.2 (A), MX211.2 (ROW)
- new net: D311.2 (A), MX311.2 (ROW)
- new net: D212.2 (A), MX212.2 (ROW)
- new net: D510.2 (A), MX510.2 (ROW)
- new net: D411.2 (A), MX411.2 (ROW)
- new net: D511.2 (A), MX511.2 (ROW)
- new net: D710.2 (A), MX710.2 (ROW)
- new net: D611.2 (A), MX611.2 (ROW)
- new net: D711.2 (A), MX711.2 (ROW)
- new net: D612.2 (A), MX612.2 (ROW)
- new net: D910.2 (A), MX910.2 (ROW)
- new net: D911.2 (A), MX911.2 (ROW)
