File: railroad-keyboard.kicad_pcb (KiCad board)
At the start: 2 copper layers, 452.4 x 104.8 mm, 214 parts, among them J1 1734510-1, SW1 SW_Push, U1 ATmega32U4-AU, U2 TRRS, Y1 16MHz

Commit message: Start reworking routing again
Parts:
- added REF**: MountingHole_2.2mm_M2, MountingHole:MountingHole_2.2mm_M2, F.Cu at (192.9, 304.8)
- added REF**: MountingHole_2.2mm_M2, MountingHole:MountingHole_2.2mm_M2, F.Cu at (254.8, 278.8)
- R2, R3: moved to F.Cu
- moved C7 37.7 mm to (175.5, 281.3)
- moved C4 34.8 mm to (178.5, 281.2)
- moved R1 13.1 mm to (184.3, 269.5), turned to 0 degrees
- moved D410 12.6 mm to (435.8, 290.4), turned to 90 degrees
- moved R6 11.3 mm to (196.2, 285.5), turned to 180 degrees
- moved R5 8.33 mm to (185.6, 239.1)
- moved C8 7.76 mm to (186.9, 242.7)
- moved F1 3.73 mm to (189.3, 248.5), turned to 90 degrees
- moved C5 3.60 mm to (181.6, 281.3), turned to 90 degrees
- moved R3 2.81 mm to (191.7, 249.1)
- moved SW1 2.41 mm to (19.1, 240.8)
- moved D304 2.10 mm to (213.2, 273.0)
- moved D504 2.10 mm to (213.0, 292.0)
- moved R2 1.78 mm to (194.1, 249.1)
- moved D702 1.61 mm to (126.4, 311.1)
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Connections:
- R6 pad 1: GND -> +5V
Routing:
- net LHD1: track 266.9 -> 0.00 mm, vias 2 -> 0
- net LHD0: track 266.6 -> 0.00 mm, vias 2 -> 0
- net +5V: track 350.6 -> 94.6 mm
- net COL10: track 326.9 -> 84.9 mm
- net Net-(R1-Pad2): track 225.1 -> 5.39 mm, vias 4 -> 0
- net ROW3: track 438.2 -> 225.5 mm, vias 4 -> 0
- net COL0: track 345.1 -> 151.6 mm, vias 1 -> 0
- net COL9: track 375.4 -> 196.9 mm, vias 1 -> 0
- net COL8: track 316.0 -> 175.4 mm, vias 1 -> 0
- net COL1: track 295.3 -> 184.2 mm, vias 1 -> 0
- net ROW4: track 462.7 -> 357.6 mm, vias 0 -> 2
- net COL7: track 263.8 -> 161.1 mm, vias 1 -> 0
- net ROW5: track 348.1 -> 259.1 mm
- net COL2: track 248.9 -> 181.1 mm, vias 1 -> 0
- net COL6: track 222.7 -> 158.1 mm, vias 1 -> 0
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- removed copper zone on B.Cu, net GND
