File: railroad-keyboard.kicad_pcb (KiCad board)
At the start: 2 copper layers, 452.4 x 104.8 mm, 216 parts, among them J1 1734510-1, SW1 SW_Push, U1 ATmega32U4-AU, U2 TRRS, Y1 16MHz

Commit message: Start adding plate
Parts:
- added REF**: MountingHole_2.2mm_M2, MountingHole:MountingHole_2.2mm_M2, F.Cu at (451.8, 228.5)
- added REF**: breakaway-mousebites, Keebio-Parts:breakaway-mousebites, F.Cu at (57.2, 232.4)
- added REF**: breakaway-mousebites, Keebio-Parts:breakaway-mousebites, F.Cu at (57.2, 234.8)
Other:
- board size 452.4 x 104.8 mm -> 462 x 221.7 mm
