File: railroad-keyboard-bottom-plate.kicad_pcb (KiCad board)
At the start: 2 copper layers, 462 x 116.9 mm, 14 parts

Commit message: Further progress
Parts:
- removed REF** (x14): MountingHole_2.2mm_M2, MountingHole:MountingHole_2.2mm_M2
Other:
- outline, holes or cut-outs redrawn
- board text added: "Railroad PCB W. Alex Ronke (NoPunIn10Did) Prototype 2020-07"

Commit message: Just about ready to send to JLCPCB
Parts:
- added J2: Conn_01x01, Connector_PinHeader_1.00mm:PinHeader_1x01_P1.00mm_Horizontal, F.Cu at (444.5, 127.0)
Routing:
- added copper zone on B.Cu, net GND1
- added copper zone on F.Cu, net GND1
Changed lines of the file:
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@@
     (tracks 0)
     (zones 0)
-    (modules 0)
-    (nets 1)
+    (modules 1)
+    (nets 2)
   )
   (page A4)
@@
     (visible_elements 7FFFFFFF)
     (pcbplotparams
-      (layerselection 0x010fc_ffffffff)
+      (layerselection 0x011fc_ffffffff)
       (usegerberextensions false)
       (usegerberattributes true)
@@
       (outputformat 1)
       (mirror false)
-      (drillshape 1)
+      (drillshape 0)
       (scaleselection 1)
-      (outputdirectory ""))
+      (outputdirectory "gerber/bottom-plate/"))
   )
   (net 0 "")
+  (net 1 GND1)
   (net_class Default "This is the default net class."
     (clearance 0.2)
@@
     (uvia_dia 0.3)
     (uvia_drill 0.1)
+    (add_net GND1)
   )
   (net_class "Net Power" ""
@@
     (uvia_drill 0.1)
   )
+  (module Connector_PinHeader_1.00mm:PinHeader_1x01_P1.00mm_Horizontal (layer F.Cu)
+    (at 444.5 127)
+    (descr "Through hole angled pin header, 1x01, 1.00mm pitch, 2.0mm pin length, single row")
+    (tags "Through hole angled pin header THT 1x01 1.00mm single row")
+    (fp_text reference J2 (at 1.375 -1.5) (layer F.SilkS)
+      (effects (font (size 1 1) (thickness 0.15)))
+    )
+    (fp_text value Conn_01x01 (at 1.375 1.5) (layer F.Fab)
+      (effects (font (size 1 1) (thickness 0.15)))
+    )
+    (fp_line (start 0.5 -0.5) (end 1.25 -0.5) (layer F.Fab) (width 0.1))
+    (fp_line (start 1.25 -0.5) (end 1.25 0.5) (layer F.Fab) (width 0.1))
+    (fp_line (start 1.25 0.5) (end 0.25 0.5) (layer F.Fab) (width 0.1))
+    (fp_line (start 0.25 0.5) (end 0.25 -0.25) (layer F.Fab) (width 0.1))
+    (fp_line (start 0.25 -0.25) (end 0.5 -0.5) (layer F.Fab) (width 0.1))
+    (fp_line (start -0.15 -0.15) (end 0.25 -0.15) (layer F.Fab) (width 0.1))
+    (fp_line (start -0.15 -0.15) (end -0.15 0.15) (layer F.Fab) (width 0.1))
+    (fp_line (start -0.15 0.15) (end 0.25 0.15) (layer F.Fab) (width 0.1))
+    (fp_line (start 1.25 -0.15) (end 3.25 -0.15) (layer F.Fab) (width 0.1))
+    (fp_line (start 3.25 -0.15) (end 3.25 0.15) (layer F.Fab) (width 0.1))
+    (fp_line (start 1.25 0.15) (end 3.25 0.15) (layer F.Fab) (width 0.1))
+    (fp_line (start 0.685 -0.56) (end 1.31 -0.56) (layer F.SilkS) (width 0.12))
+    (fp_line (start 1.31 -0.56) (end 1.31 0.56) (layer F.SilkS) (width 0.12))
+    (fp_line (start 1.31 0.56) (end 0.685 0.56) (layer F.SilkS) (width 0.12))
+    (fp_line (start 1.31 -0.21) (end 3.31 -0.21) (layer F.SilkS) (width 0.12))
+    (fp_line (start 3.31 -0.21) (end 3.31 0.21) (layer F.SilkS) (width 0.12))
+    (fp_line (start 3.31 0.21) (end 1.31 0.21) (layer F.SilkS) (width 0.12))
+    (fp_line (start 1.31 -0.15) (end 3.31 -0.15) (layer F.SilkS) (width 0.12))
+    (fp_line (start 1.31 -0.03) (end 3.31 -0.03) (layer F.SilkS) (width 0.12))
+    (fp_line (start 1.31 0.09) (end 3.31 0.09) (layer F.SilkS) (width 0.12))
+    (fp_line (start -0.685 0) (end -0.685 -0.685) (layer F.SilkS) (width 0.12))
+    (fp_line (start -0.685 -0.685) (end 0 -0.685) (layer F.SilkS) (width 0.12))
+    (fp_line (start -1 -1) (end -1 1) (layer F.CrtYd) (width 0.05))
+    (fp_line (start -1 1) (end 3.75 1) (layer F.CrtYd) (width 0.05))
+    (fp_line (start 3.75 1) (end 3.75 -1) (layer F.CrtYd) (width 0.05))
+    (fp_line (start 3.75 -1) (end -1 -1) (layer F.CrtYd) (width 0.05))
+    (fp_text user %R (at 0.75 0 90) (layer F.Fab)
+      (effects (font (size 0.6 0.6) (thickness 0.09)))
+    )
+    (pad 1 thru_hole rect (at 0 0) (size 0.85 0.85) (drill 0.5) (layers *.Cu *.Mask)
+      (net 1 GND1))
+    (model ${KISYS3DMOD}/Connector_PinHeader_1.00mm.3dshapes/PinHeader_1x01_P1.00mm_Horizontal.wrl
+      (at (xyz 0 0 0))
+      (scale (xyz 1 1 1))
+      (rotate (xyz 0 0 0))
+    )
+  )
   (gr_curve (pts (xy 287.117 180.491) (xy 286.927 180.791) (xy 287.087 180.851) (xy 288.627 181.051)) (layer B.SilkS) (width 0.5))
   (gr_curve (pts (xy 271.257 181.771) (xy 271.737001 182.121) (xy 272.077 182.151) (xy 272.227 181.871)) (layer B.SilkS) (width 0.5))
@@
   (gr_line (start -8.4074 113.64595) (end -8.4074 229.00005) (layer Edge.Cuts) (width 0.2))
   (gr_arc (start -7.61365 113.64595) (end -7.61365 112.8522) (angle -90) (layer Edge.Cuts) (width 0.2))
+  (zone (net 1) (net_name GND1) (layer F.Cu) (hatch edge 0.508)
+    (connect_pads (clearance 0.508))
+    (min_thickness 0.254)
+    (fill yes (arc_segments 32) (thermal_gap 0.508) (thermal_bridge_width 0.508))
+    (polygon
+      (pts
+        (xy 453.517 113.411) (xy 453.517 229.108) (xy 452.882 229.743) (xy -7.747 229.743) (xy -8.382 229.108)
+        (xy -8.382 113.411) (xy -7.747 112.903) (xy 452.882 112.903)
+      )
+    )
+  )
+  (zone (net 1) (net_name GND1) (layer B.Cu) (hatch edge 0.508)
+    (connect_pads (clearance 0.508))
+    (min_thickness 0.254)
+    (fill yes (arc_segments 32) (thermal_gap 0.508) (thermal_bridge_width 0.508))
+    (polygon
+      (pts
+        (xy 453.517 113.538) (xy 453.517 229.108) (xy 452.755 229.743) (xy -7.62 229.743) (xy -8.382 229.108)
+        (xy -8.382 113.538) (xy -7.62 112.903) (xy 452.882 112.903)
+      )
+    )
+  )
 )
