File: railroad-keyboard-switch-plate.kicad_pcb (KiCad board)
At the start: 2 copper layers, 462 x 116.9 mm, 14 parts

Commit message: Further progress
Parts:
- removed REF** (x14): MountingHole_2.2mm_M2, MountingHole:MountingHole_2.2mm_M2
Other:
- outline, holes or cut-outs redrawn
- board text added: "Railroad PCB W. Alex Ronke (NoPunIn10Did) Prototype 2020-07"

Commit message: Just about ready to send to JLCPCB
Parts:
- added J3: Conn_01x01, Connector_PinHeader_1.00mm:PinHeader_1x01_P1.00mm_Horizontal, F.Cu at (21.2, 396.6)
Routing:
- added copper zone on B.Cu, net GND2
- added copper zone on F.Cu, net GND2
Other:
- outline, holes or cut-outs redrawn
