File: railroad-keyboard-pcb-only.kicad_pcb (KiCad board)
At the start: 2 copper layers, 463 x 349.5 mm, 217 parts, among them J1 1734510-1, SW1 SW_Push, U1 ATmega32U4-AU, U2 TRRS, Y1 16MHz

Commit message: Just about ready to send to JLCPCB
Routing:
- added copper zone on F.Cu, net GND
Other:
- board size 463 x 349.5 mm -> 448.5 x 103 mm

Commit message: Needed some changes
Parts:
- R2, R3: moved to B.Cu
- moved R3 1.92 mm to (191.9, 251.0)
- moved R2 1.91 mm to (194.1, 251.0)
Routing:
- net D-: track 6.42 -> 8.42 mm, vias 0 -> 1
- net Net-(R2-Pad1): track 32.1 -> 30.2 mm, vias 1 -> 2
- net D+: track 3.89 -> 5.78 mm, vias 0 -> 1
- net Net-(R3-Pad1): track 31.4 -> 29.6 mm, vias 1 -> 2
