File: railroad-keyboard-pcb-only.kicad_pcb (KiCad board)
At the start: 2 copper layers, 448.5 x 103 mm, 217 parts, among them J1 1734510-1, SW1 SW_Push, U1 ATmega32U4-AU, U2 TRRS, Y1 16MHz

Commit message: Update Reset Switch and routing
Parts:
- SW1: footprint random-keyboard-parts:SKQG-1155865 -> Keebio-Parts:SW_Tactile_SPST_Angled_MJTP1117
- moved R7 29.2 mm to (405.9, 250.6), turned to 90 degrees
- moved R8 25.9 mm to (408.6, 250.6), turned to 90 degrees
- moved D10 6.24 mm to (440.7, 252.7)
- moved D104 5.61 mm to (207.4, 253.5)
- moved R5 2.22 mm to (186.8, 242.7), turned to 270 degrees
- moved SW1 1.83 mm to (20.9, 240.9), turned to 180 degrees
- moved C3 1.65 mm to (181.6, 277.8)
- moved U2 1.14 mm to (428.6, 239.3)
- moved D109 1.08 mm to (413.1, 255.0)
- moved D9 0.92 mm to (393.6, 251.6)
- moved R1 0.89 mm to (184.4, 270.4), turned to 90 degrees
- moved F1 0.67 mm to (188.6, 248.5)
- moved D106 0.57 mm to (288.3, 253.5)
- moved D108 0.45 mm to (364.5, 253.5)
- moved D105 0.44 mm to (245.5, 253.5)
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Routing:
- net GND: track 555.6 -> 588.9 mm, vias 7 -> 8
- net LHD0: track 266.5 -> 285.6 mm
- net LHD1: track 264.5 -> 282.9 mm
- net VCC: track 261.0 -> 250.4 mm
- net COL9: track 393.1 -> 401.1 mm
- net Net-(R1-Pad2): track 199.9 -> 207.3 mm
- net ROW0: track 440.6 -> 446.9 mm
- net +5V: track 95.4 -> 90.6 mm, vias 6 -> 3
- net Net-(D109-Pad2): track 7.54 -> 3.69 mm
- net Net-(D104-Pad2): track 12.6 -> 9.30 mm
- net Net-(C8-Pad2): track 14.1 -> 11.3 mm
- net COL8: track 329.4 -> 331.5 mm
- net COL0: track 390.4 -> 392.3 mm
- net COL7: track 277.6 -> 279.5 mm
- net COL1: track 308.2 -> 306.3 mm
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