File: railroad-junction/railroad-junction.kicad_pcb (KiCad board)
At the start: 2 copper layers, 128 parts, among them SW1 SW_Push, U1 TRRS

Commit message: Update to the symmetric switch libraries
Parts:
- removed MX281_100, MX291_100: MX-NoLED, railroad-junction:MXOnly-1U-Symmetric
- moved MX170_200 316.8 mm to (165.1, 36.5)
- moved MX190_200 268.3 mm to (184.2, 36.5)
- moved MX271_150 239.8 mm to (160.3, 55.6)
- moved MX291_150 177.7 mm to (188.9, 55.6)
- moved MX372_175 159.5 mm to (162.7, 74.6), turned to 180 degrees
- turned MX170_100 to 180 degrees
- turned MX180 to 180 degrees
- turned MX190_100 to 180 degrees
- turned MX271_100 to 180 degrees
