File: railroad-junction/railroad-junction.sch (KiCad schematic (older format))
At the start: 15 parts

Commit message: Sketch up split railroad
Parts:
- removed MX110_125, MX110_ISO, MX140_175, MX140_275: MX-NoLED, symbol MX_Alps_Hybrid:MX-NoLED
- added D120, D150, D160, D170, D180, D190, D211, D221, D231, D241, D251, D261, D271, D281, D291, D302, D312, D322, D332, D342, D352, D362, D372, D382, D392, D403, D413, D423, D433, D443, D453, D463, D473, D483, D493, D504, D514, D524, D544, D554, D564, D574, D584, D594: D_Small, symbol Device:D_Small
- added D_LH_100: D_Small_ALT, symbol Device:D_Small_ALT
- added MX110, MX120, MX140, MX150, MX160, MX170_100, MX170_200, MX180, MX190_100, MX190_200, MX201_150, MX201_IS0, MX211, MX221, MX231, MX241, MX251, MX261, MX271_100, MX271_150, MX281_100, MX281_175, MX291_100, MX291_150, MX302_125, MX302_150, MX312, MX322, MX332, MX342, MX352, MX362, MX372_100, MX372_175, MX382_100, MX382_175, MX382_225, MX392_100, MX392_101, MX403, MX413_100, MX413_200, MX413_225, MX423, MX433, MX443, MX453, MX463, MX473_100, MX473_175, MX483_100, MX483_225, MX483_275, MX493_100, MX493_101, MX493_175, MX504_175, MX504_275, MX514, MX524_100, MX524_125, MX544, MX554, MX564, MX574_100, MX574_125, MX574_150, MX584_100, MX584_125, MX584_150, MX594_100, MX594_125, MX594_150: MX-NoLED, symbol MX_Alps_Hybrid:MX-NoLED
- added U_RH_1: ProMicro, symbol keebio:ProMicro
- gave numbers to parts that had none: 1
- renumbered D100 to D201, MX100_150 to MX201_125
Connections:
- net Col0: now also MX201_125.1 (COL), D_LH_100.2 (A), MX201_150.1 (COL), MX201_IS0.1 (COL), MX302_125.1 (COL), MX302_150.1 (COL), MX403.1 (COL), MX504_175.1 (COL), U_RH_1.11 (8/PB4)
- net Col1: now also MX110.1 (COL), MX211.1 (COL), MX312.1 (COL), MX413_100.1 (COL), MX413_200.1 (COL), MX413_225.1 (COL), MX514.1 (COL), U_RH_1.12 (9/PB5)
- net Col2: now also MX120.1 (COL), MX221.1 (COL), MX322.1 (COL), MX423.1 (COL), MX524_100.1 (COL), MX524_125.1 (COL), U_RH_1.13 (10/PB6)
- net Col3: now also MX130.1 (COL), MX231.1 (COL), MX332.1 (COL), MX433.1 (COL), U_RH_1.14 (16/PB2)
- net Col4: now also MX140.1 (COL), MX241.1 (COL), MX342.1 (COL), MX443.1 (COL), MX544.1 (COL), U_RH_1.15 (14/PB3)
- net Col5: now also MX150.1 (COL), MX251.1 (COL), MX352.1 (COL), MX453.1 (COL), MX554.1 (COL), U_RH_1.16 (15/PB1)
- net Col6: now also MX160.1 (COL), MX261.1 (COL), MX362.1 (COL), MX463.1 (COL), MX564.1 (COL), U_RH_1.17 (A0/PF7)
- net Col7: now also MX170_100.1 (COL), MX170_200.1 (COL), MX271_100.1 (COL), MX271_150.1 (COL), MX372_100.1 (COL), MX372_175.1 (COL), MX473_100.1 (COL), MX473_175.1 (COL), MX574_100.1 (COL), MX574_125.1 (COL), MX574_150.1 (COL), U_RH_1.18 (A1/PF6)
- net Col8: now also MX180.1 (COL), MX281_100.1 (COL), MX281_175.1 (COL), MX382_100.1 (COL), MX382_175.1 (COL), MX382_225.1 (COL), MX483_100.1 (COL), MX483_225.1 (COL), MX483_275.1 (COL), MX584_100.1 (COL), MX584_125.1 (COL), MX584_150.1 (COL), U_RH_1.19 (A2/PF5)
- net Col9: now also MX190_100.1 (COL), MX190_200.1 (COL), MX291_100.1 (COL), MX291_150.1 (COL), MX392_100.1 (COL), MX392_101.1 (COL), MX493_100.1 (COL), MX493_101.1 (COL), MX493_175.1 (COL), MX594_100.1 (COL), MX594_125.1 (COL), MX594_150.1 (COL), U_RH_1.20 (A3/PF4)
- net GND: now also U_RH_1.23 (GND), U_RH_1.3 (GND), U_RH_1.4 (GND)
- net Row0: now also D110.1 (K), D130.1 (K), D140.1 (K), D120.1 (K), D150.1 (K), D160.1 (K), D170.1 (K), D180.1 (K), D190.1 (K), D_LH_100.1 (K), U_RH_1.1 (TX0/PD3)
- net Row1: now also D201.1 (K), D211.1 (K), D221.1 (K), D231.1 (K), D241.1 (K), D251.1 (K), D261.1 (K), D271.1 (K), D281.1 (K), D291.1 (K), U_RH_1.2 (RX1/PD2)
- net Row2: now also D302.1 (K), D312.1 (K), D322.1 (K), D332.1 (K), D342.1 (K), D352.1 (K), D362.1 (K), D372.1 (K), D382.1 (K), D392.1 (K), U_RH_1.7 (4/PD4)
- net Row3: now also D403.1 (K), D413.1 (K), D423.1 (K), D433.1 (K), D443.1 (K), D453.1 (K), D463.1 (K), D473.1 (K), D483.1 (K), D493.1 (K), U_RH_1.8 (5/PC6)
- net Row4: now also D504.1 (K), D514.1 (K), D524.1 (K), D544.1 (K), D554.1 (K), D564.1 (K), D574.1 (K), D584.1 (K), D594.1 (K), U_RH_1.9 (6/PD7)
- net TRRS_D0: now also U_RH_1.6 (3/PD0)
- net TRRS_D1: now also U_RH_1.5 (2/PD1)
- net VCC: now also U_RH_1.21 (VCC)
- net RESET: now reaches SW?.1, U_LH_0.22 (RST)
- net RESET: now also U_RH_1.22 (RST)
- net at D201.2 (A), MX201_125.2 (ROW): now also MX201_150.2 (ROW), MX201_IS0.2 (ROW)
- net at D110.2 (A): now also MX110.2 (ROW)
- net at D140.2 (A): now also MX140.2 (ROW)
- new net: D120.2 (A), MX120.2 (ROW)
- new net: D150.2 (A), MX150.2 (ROW)
- new net: D211.2 (A), MX211.2 (ROW)
- new net: D221.2 (A), MX221.2 (ROW)
- new net: D231.2 (A), MX231.2 (ROW)
- new net: D241.2 (A), MX241.2 (ROW)
- new net: D251.2 (A), MX251.2 (ROW)
- new net: D160.2 (A), MX160.2 (ROW)
- new net: D261.2 (A), MX261.2 (ROW)
- new net: D312.2 (A), MX312.2 (ROW)
- new net: D322.2 (A), MX322.2 (ROW)
- new net: D332.2 (A), MX332.2 (ROW)
- new net: D342.2 (A), MX342.2 (ROW)
- new net: D352.2 (A), MX352.2 (ROW)
- new net: D362.2 (A), MX362.2 (ROW)
- new net: D423.2 (A), MX423.2 (ROW)
- new net: D433.2 (A), MX433.2 (ROW)
- new net: D443.2 (A), MX443.2 (ROW)
- new net: D453.2 (A), MX453.2 (ROW)
- new net: D463.2 (A), MX463.2 (ROW)
- new net: D413.2 (A), MX413_100.2 (ROW), MX413_200.2 (ROW), MX413_225.2 (ROW)
- new net: D302.2 (A), MX302_125.2 (ROW), MX302_150.2 (ROW)
- new net: D403.2 (A), MX403.2 (ROW)
- new net: D504.2 (A), MX504_175.2 (ROW), MX504_275.2 (ROW)
- new net: D514.2 (A), MX514.2 (ROW)
- new net: D524.2 (A), MX524_100.2 (ROW), MX524_125.2 (ROW)
- new net: D544.2 (A), MX544.2 (ROW)
- new net: D554.2 (A), MX554.2 (ROW)
- new net: D564.2 (A), MX564.2 (ROW)
- new net: D170.2 (A), MX170_100.2 (ROW), MX170_200.2 (ROW)
- new net: D180.2 (A), MX180.2 (ROW)
- new net: D190.2 (A), MX190_100.2 (ROW), MX190_200.2 (ROW)
- new net: D271.2 (A), MX271_100.2 (ROW), MX271_150.2 (ROW)
- new net: D281.2 (A), MX281_100.2 (ROW), MX281_175.2 (ROW)
- new net: D291.2 (A), MX291_100.2 (ROW), MX291_150.2 (ROW)
- new net: D372.2 (A), MX372_100.2 (ROW), MX372_175.2 (ROW)
- new net: D382.2 (A), MX382_100.2 (ROW), MX382_175.2 (ROW), MX382_225.2 (ROW)
- new net: D392.2 (A), MX392_100.2 (ROW), MX392_101.2 (ROW)
- new net: D473.2 (A), MX473_100.2 (ROW), MX473_175.2 (ROW)
- new net: D483.2 (A), MX483_100.2 (ROW), MX483_225.2 (ROW), MX483_275.2 (ROW)
- new net: D493.2 (A), MX493_100.2 (ROW), MX493_101.2 (ROW), MX493_175.2 (ROW)
- new net: D574.2 (A), MX574_100.2 (ROW), MX574_125.2 (ROW), MX574_150.2 (ROW)
- new net: D584.2 (A), MX584_100.2 (ROW), MX584_125.2 (ROW), MX584_150.2 (ROW)
- new net: D594.2 (A), MX594_100.2 (ROW), MX594_125.2 (ROW), MX594_150.2 (ROW)
Other:
- moved on the sheet: D201, MX201_125, SW?

Commit message: Footprints and switch layout
Parts:
- removed MX201_IS0, MX302_125: MX-NoLED, symbol MX_Alps_Hybrid:MX-NoLED
- D110, D120, D130, D140, D150, D160, D170, D180, D190, D201, D211, D221, D231, D241, D251, D261, D271, D281, D291, D302, D312, D322, D332, D342, D352, D362, D372, D382, D392, D403, D413, D423, D433, D443, D453, D463, D473, D483, D493, D504, D514, D524, D544, D554, D564, D574, D584, D594, D_LH_100: footprint (none) -> Keebio-Parts:Diode
- MX110, MX120, MX130, MX140, MX150, MX160, MX170_100, MX180, MX190_100, MX211, MX221, MX231, MX241, MX251, MX261, MX271_100, MX281_100, MX291_100, MX312, MX322, MX332, MX342, MX352, MX362, MX372_100, MX382_100, MX392_100, MX392_101, MX403, MX413_100, MX423, MX433, MX443, MX453, MX463, MX473_100, MX483_100, MX493_100, MX493_101, MX514, MX524_100, MX544, MX554, MX564, MX574_100, MX584_100, MX594_100: footprint (none) -> railroad-junction:MXOnly-1U-Symmetric
- MX170_200, MX190_200, MX413_200: footprint (none) -> railroad-junction:MXOnly-2U-Symmetric
- MX201_125, MX524_125, MX574_125, MX584_125, MX594_125: footprint (none) -> railroad-junction:MXOnly-1.25U-Symmetric
- MX201_IS0: renamed from MX201_150; footprint (none) -> railroad-junction:MXOnly-ISO-ROTATED-ReversedStabilizers-Symmetric
- MX271_150, MX291_150, MX574_150, MX584_150, MX594_150: footprint (none) -> railroad-junction:MXOnly-1.5U-Symmetric
- MX281_175, MX372_175, MX382_175, MX473_175, MX493_175, MX504_175: footprint (none) -> railroad-junction:MXOnly-1.75U-Symmetric
- MX302_125: renamed from MX302_150; footprint (none) -> railroad-junction:MXOnly-1.25U-Symmetric
- MX382_225, MX413_225, MX483_225: footprint (none) -> railroad-junction:MXOnly-2.25U-Symmetric
- MX483_275, MX504_275: footprint (none) -> railroad-junction:MXOnly-2.75U-Symmetric
- R1, R2: renamed from R?; footprint (none) -> Keebio-Parts:Resistor
- SW1: renamed from SW?; footprint (none) -> Keebio-Parts:SW_Tactile_SPST_Angled_MJTP1117
- U1: renamed from U?; footprint (none) -> Keebio-Parts:TRRS-PJ-320A-dual
- U_LH_0, U_RH_1: footprint (none) -> Keebio-Parts:ArduinoProMicro
Other:
- moved on the sheet: MX302_125

Commit message: Update to the symmetric switch libraries
Parts:
- removed MX281_100, MX291_100: MX-NoLED, railroad-junction:MXOnly-1U-Symmetric, symbol MX_Alps_Hybrid:MX-NoLED
Changed lines of the file:
@@
 Connection ~ 7600 2150
-$Comp
-L MX_Alps_Hybrid:MX-NoLED MX281_100
-U 1 1 5F119D5B
-P 8600 1900
-F 0 "MX281_100" H 8633 2123 60  0000 C CNN
-F 1 "MX-NoLED" H 8633 2049 20  0000 C CNN
-F 2 "railroad-junction:MXOnly-1U-Symmetric" H 7975 1875 60  0001 C CNN
-F 3 "" H 7975 1875 60  0001 C CNN
-	1    8600 1900
-	1    0    0    -1
-$EndComp
 $Comp
 L Device:D_Small D281
@@
 	0    -1   -1   0
 $EndComp
-Wire Wire Line
-	8550 2050 8550 2150
 $Comp
 L MX_Alps_Hybrid:MX-NoLED MX281_175
@@
 Wire Wire Line
 	8550 2150 8550 2250
-Connection ~ 8550 2150
-$Comp
-L MX_Alps_Hybrid:MX-NoLED MX291_100
-U 1 1 5F11BA7F
-P 9550 1900
-F 0 "MX291_100" H 9583 2123 60  0000 C CNN
-F 1 "MX-NoLED" H 9583 2049 20  0000 C CNN
-F 2 "railroad-junction:MXOnly-1U-Symmetric" H 8925 1875 60  0001 C CNN
-F 3 "" H 8925 1875 60  0001 C CNN
-	1    9550 1900
-	1    0    0    -1
-$EndComp
 $Comp
 L Device:D_Small D291
@@
 	0    -1   -1   0
 $EndComp
-Wire Wire Line
-	9500 2050 9500 2150
 $Comp
 L MX_Alps_Hybrid:MX-NoLED MX291_150
@@
 Wire Wire Line
 	9500 2150 9500 2250
-Connection ~ 9500 2150
 $Comp
 L MX_Alps_Hybrid:MX-NoLED MX372_100
@@
 Connection ~ 9150 1200
 Wire Wire Line
-	9150 1200 9150 1850
-Wire Wire Line
-	8750 1850 9150 1850
-Connection ~ 9150 1850
-Wire Wire Line
-	9150 1850 9150 1950
-Wire Wire Line
 	9150 1950 9150 2700
 Wire Wire Line
@@
 	10100 1000 10100 1100
 Connection ~ 9700 1000
-Wire Wire Line
-	10100 1100 10100 1850
 Connection ~ 10100 1100
 Wire Wire Line
@@
 Wire Wire Line
 	10350 3550 10350 2800
-Wire Wire Line
-	9700 1850 10100 1850
-Connection ~ 10100 1850
-Wire Wire Line
-	10100 1850 10100 1950
 Text GLabel 1900 1700 0    50   Input ~ 0
 Row0
@@
 Wire Wire Line
 	3200 1850 3200 2850
+Wire Wire Line
+	10100 1100 10100 1950
+Wire Wire Line
+	9150 1200 9150 1950
 $EndSCHEMATC
